File: Senior_Design/Senior_Design/power_layout.brd (EAGLE design)
At the start: 105.8 x 35 mm, 57 parts, among them IC1 MIC29302WU, J1 AU-Y1008-2, J1[SIMCARD] 78646-3001, J2 U.FL-R-SMT-1(01), J4[GROVE] 640456-4, T1 BCX70SMD, T2 BCX70SMD, U1 SIM7000E, U2 TUSB2046BVFR, U3 PCA9306DQER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

Commit message: Added values to passives
Parts:
- C1: value (none) -> 100 uF
- C10, C11, C6, C8, C9: value (none) -> 0.1 uF
- C3: value (none) -> 330 uF
- C4: value (none) -> 1 uF
- C5: value (none) -> 100 nF
- R1: value (none) -> 10 ohm
- R13, R15, R9: value (none) -> 4.7k ohm
- R19, R20, R21, R22, R7, R8: value (none) -> 27 ohm
- R2, R3: value (none) -> 60 ohm
- R4: value (none) -> 47k ohm
- R5: value (none) -> 100k ohm
- R6: value (none) -> 470 ohm
