File: Senior_Design/power_layout.sch (EAGLE design)
At the start: 37 parts, among them IC1 MIC29302WU, J1[SIMCARD] 78646-3001, J2 292303-1, J3[GROVE] 640456-4, J4[GROVE] 640456-4, U1 SIM7000E, U2 TUSB2046BIRHBR, U3 PCA9306DQER

Commit message: Added a bit more detail to the modem design
Parts:
- added C10, C8, C9: (no value), capacitor-wima:C2,5-3
- added T1, T2: 2N706, transistor:2N706
- C1: value (none) -> 1uF; SPICEPREFIX (none) -> C
- C3: value (none) -> 0.1 uF
- C4: value (none) -> 100 uF
- C5: value (none) -> 330 uF
- R4: value (none) -> 47k
- R5: value (none) -> 100k
- R6: value (none) -> 470
Connections:
- new net +3V3: C9.1, U3.EN, U3.VREF2
- new net N$10: C10.2, T1.C, U1.!PWRKEY
- new net N$12: C8.2, U3.VREF1
- new net PWR: T1.B
- new net SLEEP: T2.B
- new net TP01: U1.BOOT_CFG
- new net VDD_EXT: T2.C, U1.DTR, U1.VDD_EXT
- net 0: now also C10.1, C8.1, C9.2, T1.E, T2.E, U3.GND
Other:
- moved on the sheet: U3

Commit message: Add files via upload
Schematic Reflects all changes as discussed in Sep 1st HW meeting.  Layout will begin tomorrow.
Parts:
- removed J3[GROVE]: 640456-4, 640456-4:640456-4
- added C11: (no value), rcl:C-USC0805
- added C12, C13: 27pF, rcl:C-USC0603
- added CR1: 9C-6.000MAAJ-T, Personal:9C-6.000MAAJ-T
- added GROVE1: 640456-4, 640456-4:640456-4
- added J1: AU-Y1008-2, Personal:AU-Y1008-2
- added R11, R18: 47k, SparkFun-Resistors:47KOHM-0603-1/10W-1%
- added R12, R17: 4.7k, SparkFun-Resistors:4.7KOHM-0603-1/10W-1%
- added R19, R20, R7, R8: 27, SparkFun-Resistors:RESISTOR0805
- added R21, R22: (no value), SparkFun-Resistors:RESISTOR0805
- added R23, R24: 15k, SparkFun-Resistors:RESISTOR0805
- added R25: 1.5k, SparkFun-Resistors:RESISTOR0805
- added TP1: TPPAD1-13, testpad:TPPAD1-13
- added U4: TPS2044BDR, Personal:TPS2044BDR
- added X1: 22-23-2041, con-molex:22-23-2041
- C1: value 1uF -> (none); device capacitor-wima:C2,5-3 -> rcl:C-USC0805; SPICEPREFIX C -> (none)
- C10, C2, C6, C7, C8, C9: device capacitor-wima:C2,5-3 -> rcl:C-USC0805
- C3: value 0.1 uF -> (none); device capacitor-wima:C2,5-3 -> rcl:C-USC0805
- C4: value 100 uF -> (none); device rcl:C-US025-024X044 -> rcl:C-USC0805
- C5: value 330 uF -> (none); device rcl:C-US025-024X044 -> rcl:C-USC0805
- D1: value (none) -> RED; device SparkFun-LED:LED-3MM-NO_SILK -> SparkFun-LED:LED-RED1206
- D2: value (none) -> GREEN; device SparkFun-LED:LED-3MM-NO_SILK -> SparkFun-LED:LED-GREEN1206
- D3: value (none) -> BLUE; device SparkFun-LED:LED-3MM-NO_SILK -> SparkFun-LED:LED-BLUE1206
- J2: value 292303-1 -> U.FL-R-SMT-1(01); device 292303-1:292303-1 -> Personal:U.FL-R-SMT-1(01)
- R1, R10, R14, R16, R2, R3: device SparkFun-Resistors:RESISTOR0402 -> SparkFun-Resistors:RESISTOR0805
- R13, R15: value (none) -> 15k; device SparkFun-Resistors:RESISTOR0402 -> SparkFun-Resistors:RESISTOR0805
- R4: value 47k -> (none); device SparkFun-Resistors:RESISTOR0402 -> SparkFun-Resistors:RESISTOR0805
- R5: value 100k -> (none); device SparkFun-Resistors:RESISTOR0402 -> SparkFun-Resistors:RESISTOR0805
- R6: value 470 -> (none); device SparkFun-Resistors:RESISTOR0402 -> SparkFun-Resistors:RESISTOR0805
- R9: value (none) -> 1.5k; device SparkFun-Resistors:RESISTOR0402 -> SparkFun-Resistors:1KOHM-0603-1/10W-1%
- T1, T2: value 2N706 -> BCX70SMD; device transistor:2N706 -> transistor:BCX70SMD
- U2: value TUSB2046BIRHBR -> TUSB2046BVFR; device TUSB2046B:TUSB2046BIRHBR -> Personal:TUSB2046BVFR
Connections:
- removed net +3V3: C9.1, U3.EN, U3.VREF2
- removed net GPIO_1: R3.2
- removed net GPIO_3: R1.2
- removed net N$11: R9.1, SW1.P$2
- removed net N$15: R15.1, SW3.P$2
- removed net TP01: U1.BOOT_CFG
- removed net UART_RXD: U1.RXD, U3.SDA2
- removed net UART_TXD: U1.TXD, U3.SCL2
- removed net WIFI_D+: J2.P3
- removed net WIFI_D-: J2.P2
- new net 1.8V: C9.1, U1.VDD_EXT, U3.VREF1
- new net 3.3V: C10.1, R25.2, SV1.14, U2.!EXTMEM, U2.VCC, U2.VCC_2, U3.EN, U3.VREF2, X1-1.S
- new net ANT: J2.2, U1.RF_ANT
- new net DM0: R8.1, SV1.9
- new net DP0: R7.1, SV1.11
- new net GND: C1.2, C10.2, C2.1, C3.2, C4.2, C5.2, C6.2, C7.1, C8.2, C9.2, D1.C, D2.C, D3.C, GROVE1.4, IC1.GND, J1.4, J1.8, J1[SIMCARD].GND, J2.1, J2.3, J4[GROVE].4, R10.1, R11.2, R14.1, R16.1, R18.1, R4.1, R6.1, SV1.15, SV2.15, T1.E, T2.E, U$1.P$2, U1.GND, U2.GND, U2.TSTMODE, U2.TSTPLL/48MCLK, U3.GND, U4.GND, U4.GND_2, X1-4.S
- new net I2C1_SCL: C2.2, GROVE1.1, SV2.9
- new net I2C1_SDA: GROVE1.2, SV2.11
- new net I2C2_SCL: C7.2, J4[GROVE].1
- new net I2C2_SDA: J4[GROVE].2
- new net LED1: R3.2, SV2.6
- new net LED2: R2.2, SV2.8
- new net LED3: R1.2, SV2.10
- new net N$13: U3.SCL2, X1-2.S
- new net N$16: U3.SDA2, X1-3.S
- new net N$17: R11.1, R12.2, T2.B
- new net N$18: R17.1, R18.2, T1.B
- new net N$19: R19.2, U2.DM2
- new net N$20: R20.2, U2.DP2
- new net N$21: J4[GROVE].3
- new net N$22: R21.1, U2.DP3
- new net N$23: R22.1, U2.DM3
- new net N$24: GROVE1.3
- new net N$25: U2.DP4
- new net N$26: U2.DM4
- new net N$27: U1.RXD, U3.SCL1
- new net N$28: U1.TXD, U3.SDA1
- new net OUT1: U4.OUT1
- new net OUT2: J1.1, U4.OUT2
- new net OUT3: J1.5, U4.OUT3
- new net OUT4: U4.NC
- new net OVRCUR1: U2.!OVRCUR1, U4.!OC1
- new net OVRCUR2: U2.!OVRCUR2, U4.!OC2
- new net OVRCUR3: U2.!OVRCUR3, U4.!OC3
- new net OVRCUR4: U2.!OVRCUR4, U4.NC_3
- new net PB2: R14.2, SV2.17, SW2.P$1
- new net PB3: R16.2, SV2.19, SW3.P$1
- new net PWRKEY: C8.1, SV2.3, T1.C, U1.!PWRKEY
- new net PWRON1: U2.!PWRON1, U4.!EN1
- new net PWRON2: U2.!PWRON2, U4.!EN2
- new net PWRON3: U2.!PWRON3, U4.!EN3
- new net PWRON4: U2.!PWRON4, U4.NC_2
- new net USB1_D+: J1.3, R20.1, R24.2
- new net USB1_D-: J1.2, R19.1, R23.2
- new net USB2_D+: J1.7, R13.2, R21.2
- new net USB2_D-: J1.6, R15.2, R22.2
- new net XTAL1: C12.1, CR1.1, U2.XTAL1
- new net XTAL2: R9.2, U2.XTAL2
- net +5V: now also C11.1, SW1.P$2, SW2.P$2, SW3.P$2, U4.IN1, U4.IN2; no longer C2.2, C7.2, J2.P1, J3[GROVE].1, J3[GROVE].2, J3[GROVE].3, J4[GROVE].1, J4[GROVE].2, J4[GROVE].3, R13.2, R15.2, R9.2
- net 0: now also C11.2, C12.2, C13.2, R13.1, R15.1, R23.1, R24.1, U2.BUSPWR, U2.EEDATA/GANGED, U2.GND_2; no longer C1.2, C10.1, C2.1, C3.2, C4.2, C5.2, C6.2, C7.1, C8.1, C9.2, D1.C, D2.C, D3.C, IC1.GND, J1[SIMCARD].GND, J2.P4, J3[GROVE].4, J4[GROVE].4, R10.1, R14.1, R16.1, R4.1, R6.1, T1.E, T2.E, U$1.P$2, U1.GND, U3.GND
- net MODEM_D+: now also U2.DP1
- net MODEM_D-: now also U2.DM1
- net N$10: now also R25.1, R7.2, U2.DP0; no longer C10.2, T1.C, U1.!PWRKEY
- net N$12: now also R8.2, U2.DM0; no longer C8.2, U3.VREF1
- net N$14: now also C13.1, CR1.2, R9.1; no longer R13.1, SW2.P$2
- net N$9: now also TP1.TP, U1.BOOT_CFG; no longer R2.2
- net NRESET: now also SV2.4; no longer R14.2, R16.2, SW2.P$1, SW3.P$1
- net PWR: now also R17.2; no longer T1.B
- net SLEEP: now also R12.1; no longer T2.B
- net VDD_EXT: no longer U1.VDD_EXT
Other:
- moved on the sheet: BRD1, C10, C6, C8, C9, J1[SIMCARD], SV1, SV2, T1, T2, U1, U3

Commit message: Add files via upload
Another push inbound
Parts:
- added C14, C15: 27pF, rcl:C-USC0603
- added D4: Yellow, SparkFun-LED:LED-YELLOW0603
- added R26, R27: 0, SparkFun-Resistors:1KOHM-0603-1/10W-1%
- added R28: 330, SparkFun-Resistors:1KOHM-0603-1/10W-1%
- added TP2: TPTP16R, testpad:TPTP16R
- R1, R2, R3: value (none) -> 330
- TP1: value TPPAD1-13 -> TPTP10R; device testpad:TPPAD1-13 -> testpad:TPTP10R
- X1: value 22-23-2041 -> 332-04; device con-molex:22-23-2041 -> con-garry:332-04
Connections:
- net VBAT renamed MODEM_POWER
- removed net 0: C11.2, C12.2, C13.2, R13.1, R15.1, R23.1, R24.1, U2.BUSPWR, U2.EEDATA/GANGED, U2.GND_2
- removed net ANT: J2.2, U1.RF_ANT
- new net N$11: C14.1, R26.1, R27.2
- new net N$15: TP2.TP, U1.GNSS_ANT
- new net N$29: R28.2, U1.NETLIGHT
- new net N$30: D4.A, R28.1
- new net PRE_ANT: C15.1, R26.2, U1.RF_ANT
- new net RF_ANT: J2.2, R27.1
- net GND: now also C11.2, C12.2, C13.2, C14.2, C15.2, D4.C, R13.1, R15.1, R23.1, R24.1, U2.BUSPWR, U2.EEDATA/GANGED, U2.GND_2
- net NRESET: no longer SV2.4
- net SLEEP: now also SV2.2
Other:
- moved on the sheet: BRD1, C10, C11, C12, C13, C6, C8, C9, CR1, J1, J1[SIMCARD], J2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

Commit message: Add files via upload
Nightly progress pre-CDR
-Still finishing Layout
~2 hours of layout left until first draft complete
Connections:
- removed net N$21: J4[GROVE].3
- removed net N$24: GROVE1.3
- removed net PWR: R17.2
- net +5V: now also GROVE1.3, J4[GROVE].3, SV1.24
- net 3.3V: now also R17.2
- net I2C2_SCL: now also SV1.28
- net I2C2_SDA: now also SV1.26
Changed lines of the file:
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@@
 <pinref part="P+3" gate="1" pin="+5V"/>
+</segment>
+<segment>
+<pinref part="SV1" gate="G$1" pin="24"/>
+<wire x1="20.32" y1="-125.73" x2="20.32" y2="-128.27" width="0.1524" layer="91"/>
+<label x="20.32" y="-128.27" size="1.778" layer="95" rot="R270" xref="yes"/>
 </segment>
 </net>
@@
 <label x="-26.67" y="142.24" size="1.778" layer="95" xref="yes" grouprefs="USB"/>
 </segment>
+<segment>
+<pinref part="R17" gate="G$1" pin="2"/>
+<wire x1="25.4" y1="41.91" x2="25.4" y2="49.53" width="0.1524" layer="91" grouprefs="SIM7000"/>
+<label x="25.4" y="49.53" size="1.778" layer="95" rot="R90" xref="yes" grouprefs="SIM7000"/>
+</segment>
 </net>
 <net name="VDD_EXT" class="0">
@@
 </segment>
 </net>
-<net name="PWR" class="0">
-<segment>
-<pinref part="R17" gate="G$1" pin="2"/>
-<wire x1="25.4" y1="41.91" x2="25.4" y2="49.53" width="0.1524" layer="91" grouprefs="SIM7000"/>
-<label x="25.4" y="49.53" size="1.778" layer="95" rot="R90" xref="yes" grouprefs="SIM7000"/>
-</segment>
-</net>
 <net name="N$18" class="0">
 <segment>
@@
 <pinref part="R28" gate="G$1" pin="1"/>
 <pinref part="D4" gate="G$1" pin="A"/>
+</segment>
+</net>
+<net name="I2C2_SDA" class="0">
+<segment>
+<pinref part="SV1" gate="G$1" pin="26"/>
+<wire x1="17.78" y1="-125.73" x2="17.78" y2="-128.27" width="0.1524" layer="91"/>
+<label x="17.78" y="-128.27" size="1.778" layer="95" rot="R270" xref="yes"/>
+</segment>
+</net>
+<net name="I2C2_SCL" class="0">
+<segment>
+<pinref part="SV1" gate="G$1" pin="28"/>
+<wire x1="15.24" y1="-125.73" x2="15.24" y2="-128.27" width="0.1524" layer="91"/>
+<label x="15.24" y="-128.27" size="1.778" layer="95" rot="R270" xref="yes"/>
 </segment>
 </net>
@@
 <pinref part="P+1" gate="1" pin="+5V"/>
 <wire x1="2.54" y1="33.02" x2="2.54" y2="35.56" width="0.1524" layer="91" grouprefs="POWER"/>
+<label x="5.08" y="38.1" size="1.778" layer="95" xref="yes"/>
 </segment>
 <segment>
@@
 <wire x1="55.88" y1="101.6" x2="55.88" y2="91.44" width="0.1524" layer="91"/>
 </segment>
-</net>
-<net name="LED3" class="0">
-<segment>
-<pinref part="R1" gate="G$1" pin="2"/>
-<wire x1="109.22" y1="91.44" x2="109.22" y2="93.98" width="0.1524" layer="91" grouprefs="USER_IO"/>
-<label x="109.22" y="93.98" size="1.778" layer="95" rot="R90" xref="yes" grouprefs="USER_IO"/>
-</segment>
-</net>
-<net name="LED1" class="0">
-<segment>
-<pinref part="R3" gate="G$1" pin="2"/>
-<wire x1="88.9" y1="91.44" x2="88.9" y2="93.98" width="0.1524" layer="91" grouprefs="USER_IO"/>
-<label x="88.9" y="93.98" size="1.778" layer="95" rot="R90" xref="yes" grouprefs="USER_IO"/>
-</segment>
-</net>
-<net name="N$8" class="0">
-<segment>
-<pinref part="D1" gate="G$1" pin="A"/>
-<pinref part="R3" gate="G$1" pin="1"/>
-</segment>
-</net>
-<net name="N$7" class="0">
-<segment>
-<pinref part="D2" gate="G$1" pin="A"/>
-<pinref part="R2" gate="G$1" pin="1"/>
-</segment>
-</net>
-<net name="LED2" class="0">
-<segment>
-<pinref part="R2" gate="G$1" pin="2"/>
-<wire x1="99.06" y1="91.44" x2="99.06" y2="93.98" width="0.1524" layer="91"/>
-<label x="99.06" y="93.98" size="1.778" layer="95" rot="R90" xref="yes"/>
-</segment>
-</net>
-<net name="N$5" class="0">
-<segment>
-<pinref part="R1" gate="G$1" pin="1"/>
-<pinref part="D3" gate="G$1" pin="A"/>
-</segment>
-</net>
-<net name="N$21" class="0">
+<segment>
+<pinref part="GROVE1" gate="G$1" pin="3"/>
+<wire x1="133.35" y1="73.66" x2="125.73" y2="73.66" width="0.1524" layer="91" grouprefs="GROVE"/>
+<wire x1="125.73" y1="86.36" x2="125.73" y2="73.66" width="0.1524" layer="91" grouprefs="GROVE"/>
+<label x="125.73" y="86.36" size="1.778" layer="95" rot="R90" xref="yes" grouprefs="GROVE"/>
+</segment>
 <segment>
 <pinref part="J4[GROVE]" gate="G$1" pin="3"/>
@@
 </segment>
 </net>
+<net name="LED3" class="0">
+<segment>
+<pinref part="R1" gate="G$1" pin="2"/>
+<wire x1="109.22" y1="91.44" x2="109.22" y2="93.98" width="0.1524" layer="91" grouprefs="USER_IO"/>
+<label x="109.22" y="93.98" size="1.778" layer="95" rot="R90" xref="yes" grouprefs="USER_IO"/>
+</segment>
+</net>
+<net name="LED1" class="0">
+<segment>
+<pinref part="R3" gate="G$1" pin="2"/>
+<wire x1="88.9" y1="91.44" x2="88.9" y2="93.98" width="0.1524" layer="91" grouprefs="USER_IO"/>
+<label x="88.9" y="93.98" size="1.778" layer="95" rot="R90" xref="yes" grouprefs="USER_IO"/>
+</segment>
+</net>
+<net name="N$8" class="0">
+<segment>
+<pinref part="D1" gate="G$1" pin="A"/>
+<pinref part="R3" gate="G$1" pin="1"/>
+</segment>
+</net>
+<net name="N$7" class="0">
+<segment>
+<pinref part="D2" gate="G$1" pin="A"/>
+<pinref part="R2" gate="G$1" pin="1"/>
+</segment>
+</net>
+<net name="LED2" class="0">
+<segment>
+<pinref part="R2" gate="G$1" pin="2"/>
+<wire x1="99.06" y1="91.44" x2="99.06" y2="93.98" width="0.1524" layer="91"/>
+<label x="99.06" y="93.98" size="1.778" layer="95" rot="R90" xref="yes"/>
+</segment>
+</net>
+<net name="N$5" class="0">
+<segment>
+<pinref part="R1" gate="G$1" pin="1"/>
+<pinref part="D3" gate="G$1" pin="A"/>
+</segment>
+</net>
 <net name="I2C2_SDA" class="0">
 <segment>
@@
 </segment>
 </net>
-<net name="N$24" class="0">
-<segment>
-<pinref part="GROVE1" gate="G$1" pin="3"/>
-<wire x1="133.35" y1="73.66" x2="125.73" y2="73.66" width="0.1524" layer="91" grouprefs="GROVE"/>
-<wire x1="125.73" y1="86.36" x2="125.73" y2="73.66" width="0.1524" layer="91" grouprefs="GROVE"/>
-<label x="125.73" y="86.36" size="1.778" layer="95" rot="R90" xref="yes" grouprefs="GROVE"/>
-</segment>
-</net>

Commit message: Add files via upload
Final Design files prior to CDR!
Includes schematic and layout
-Needs final review prior to ordering
Parts:
- added TP3, TP4, TP5, TP6: TPTP10R, testpad:TPTP10R
Connections:
- net +5V: now also TP6.TP
- net MODEM_POWER: now also TP5.TP
- net OUT2: now also TP3.TP
- net OUT3: now also TP4.TP
Other:
- moved on the sheet: BRD1, C10, C12, C13, C14, C15, C6, C8, C9, CR1, J1[SIMCARD], J2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

Commit message: Added Pre-PCB Review Changes
Polishing of post-CDR design
Parts:
- added R29, R30, R31, R32: 4700, SparkFun-Resistors:RESISTOR0805
- added R33: 220k, SparkFun-Resistors:4.7KOHM-0603-1/10W-1%
- added SJ1: (no value), jumper:SJW
Connections:
- new net N$21: R33.2, U3.EN, U3.VREF2
- net +5V: now also IC1.EN; no longer GROVE1.3, J4[GROVE].3
- net 3.3V: now also GROVE1.3, J4[GROVE].3, R29.2, R30.2, R31.2, R32.2, R33.1, SJ1.1; no longer U3.EN, U3.VREF2
- net I2C1_SCL: now also R29.1
- net I2C1_SDA: now also R30.1
- net I2C2_SCL: now also R31.1
- net I2C2_SDA: now also R32.1
- net MODEM_POWER: now also SJ1.2
