File: Senior_Design/power_layout.sch (EAGLE design)
At the start: 29 parts, among them IC1 MIC29302WU, J1 78646-3001, J2 292303-1, J3 640456-4, SW1 CT10-XXXX-A2, U1 SIM7000E

Commit message: Arthur's 1st Push
Annotated on Readme as 4/4/2020 11AM push
Parts:
- added BRD1: POCKETBEAGLE_BRD_2, e14_BeagleBoard_PocketBeagle_v1_alpha1:POCKETBEAGLE_BRD_2
- renumbered J1 to J1[SIMCARD], J3 to J3[GROVE]
Changed lines of the file:
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@@
 <?xml version="1.0" encoding="utf-8"?>
 <!DOCTYPE eagle SYSTEM "eagle.dtd">
-<eagle version="9.6.0">
+<eagle version="9.5.2">
 <drawing>
 <settings>
@@
 <layers>
 <layer number="1" name="Top" color="4" fill="1" visible="no" active="no"/>
+<layer number="2" name="Route2" color="1" fill="3" visible="no" active="no"/>
+<layer number="3" name="Route3" color="4" fill="3" visible="no" active="no"/>
+<layer number="4" name="Route4" color="1" fill="4" visible="no" active="no"/>
+<layer number="5" name="Route5" color="4" fill="4" visible="no" active="no"/>
+<layer number="6" name="Route6" color="1" fill="8" visible="no" active="no"/>
+<layer number="7" name="Route7" color="4" fill="8" visible="no" active="no"/>
+<layer number="8" name="Route8" color="1" fill="2" visible="no" active="no"/>
+<layer number="9" name="Route9" color="4" fill="2" visible="no" active="no"/>
+<layer number="10" name="Route10" color="1" fill="7" visible="no" active="no"/>
+<layer number="11" name="Route11" color="4" fill="7" visible="no" active="no"/>
+<layer number="12" name="Route12" color="1" fill="5" visible="no" active="no"/>
+<layer number="13" name="Route13" color="4" fill="5" visible="no" active="no"/>
+<layer number="14" name="Route14" color="1" fill="6" visible="no" active="no"/>
+<layer number="15" name="Route15" color="4" fill="6" visible="no" active="no"/>
 <layer number="16" name="Bottom" color="1" fill="1" visible="no" active="no"/>
 <layer number="17" name="Pads" color="2" fill="1" visible="no" active="no"/>
@@
 <part name="U1" library="SIM7000E" deviceset="SIM7000E" device=""/>
 <part name="X_8" library="ngspice-simulation" library_urn="urn:adsk.eagle:library:527439" deviceset="GND" device=""/>
-<part name="J1" library="78646-3001" deviceset="78646-3001" device=""/>
+<part name="J1[SIMCARD]" library="78646-3001" deviceset="78646-3001" device=""/>
 <part name="X_9" library="ngspice-simulation" library_urn="urn:adsk.eagle:library:527439" deviceset="GND" device=""/>
 <part name="D1" library="SparkFun-LED" library_urn="urn:adsk.eagle:library:529" deviceset="LED" device="-3MM-NO_SILK" package3d_urn="urn:adsk.eagle:package:39356/1"/>
@@
 <part name="X_13" library="ngspice-simulation" library_urn="urn:adsk.eagle:library:527439" deviceset="GND" device=""/>
 <part name="P+2" library="supply1" library_urn="urn:adsk.eagle:library:371" deviceset="+5V" device=""/>
-<part name="J3" library="640456-4" deviceset="640456-4" device=""/>
+<part name="J3[GROVE]" library="640456-4" deviceset="640456-4" device=""/>
 <part name="R1" library="SparkFun-Resistors" library_urn="urn:adsk.eagle:library:532" deviceset="RESISTOR" device="0402" package3d_urn="urn:adsk.eagle:package:39657/1" value=" "/>
 <part name="R2" library="SparkFun-Resistors" library_urn="urn:adsk.eagle:library:532" deviceset="RESISTOR" device="0402" package3d_urn="urn:adsk.eagle:package:39657/1" value=" "/>
@@
 <part name="X_20" library="ngspice-simulation" library_urn="urn:adsk.eagle:library:527439" deviceset="GND" device=""/>
 <part name="X_21" library="ngspice-simulation" library_urn="urn:adsk.eagle:library:527439" deviceset="GND" device=""/>
+<part name="BRD1" library="e14_BeagleBoard_PocketBeagle_v1_alpha1" deviceset="POCKETBEAGLE_?_2" device="BRD"/>
 </parts>
 <sheets>
@@
 </instance>
 <instance part="X_8" gate="G$1" x="88.9" y="-40.64" smashed="yes" rot="MR0"/>
-<instance part="J1" gate="G$1" x="134.62" y="12.7" smashed="yes">
+<instance part="J1[SIMCARD]" gate="G$1" x="134.62" y="12.7" smashed="yes">
 <attribute name="NAME" x="127.4986" y="23.3776" size="1.780359375" layer="95"/>
 <attribute name="VALUE" x="127.22353125" y="-2.084" size="1.78643125" layer="96"/>
@@
 <attribute name="VALUE" x="149.86" y="60.96" size="1.778" layer="96" rot="R90"/>
 </instance>
-<instance part="J3" gate="G$1" x="200.66" y="15.24" smashed="yes">
+<instance part="J3[GROVE]" gate="G$1" x="200.66" y="15.24" smashed="yes">
 <attribute name="NAME" x="195.08" y="22.86" size="1.778" layer="95"/>
 <attribute name="VALUE" x="195.58" y="7.62" size="1.778" layer="96"/>
@@
 <instance part="X_20" gate="G$1" x="93.98" y="-5.08" smashed="yes" rot="MR0"/>
 <instance part="X_21" gate="G$1" x="111.76" y="-5.08" smashed="yes" rot="MR0"/>
+<instance part="BRD1" gate="G$1" x="-175.26" y="15.24" smashed="yes">
+<attribute name="NAME" x="-162.56" y="93.98" size="1.778" layer="95" align="center-left"/>
+<attribute name="VALUE" x="-162.56" y="91.44" size="1.778" layer="96" align="center-left"/>
+</instance>
 </instances>
 <busses>
@@
 </segment>
 <segment>
-<pinref part="J1" gate="G$1" pin="GND"/>
+<pinref part="J1[SIMCARD]" gate="G$1" pin="GND"/>
 <wire x1="147.32" y1="2.54" x2="152.4" y2="2.54" width="0.1524" layer="91"/>
 <wire x1="152.4" y1="2.54" x2="152.4" y2="-2.54" width="0.1524" layer="91"/>
@@
 </segment>
 <segment>
-<pinref part="J3" gate="G$1" pin="4"/>
+<pinref part="J3[GROVE]" gate="G$1" pin="4"/>
 <wire x1="190.5" y1="12.7" x2="190.5" y2="10.16" width="0.1524" layer="91"/>
 <pinref part="X_14" gate="G$1" pin="0"/>
@@
 <pinref part="U1" gate="G$1" pin="SIM_CLK"/>
 <wire x1="86.36" y1="12.7" x2="121.92" y2="12.7" width="0.1524" layer="91"/>
-<pinref part="J1" gate="G$1" pin="RST"/>
+<pinref part="J1[SIMCARD]" gate="G$1" pin="RST"/>
 </segment>
 </net>
@@
 <pinref part="U1" gate="G$1" pin="SIM_RST"/>
 <wire x1="86.36" y1="10.16" x2="109.22" y2="10.16" width="0.1524" layer="91"/>
-<pinref part="J1" gate="G$1" pin="CLK"/>
+<pinref part="J1[SIMCARD]" gate="G$1" pin="CLK"/>
 <pinref part="D5" gate="1" pin="C"/>
 <wire x1="109.22" y1="10.16" x2="111.76" y2="10.16" width="0.1524" layer="91"/>
@@
 <wire x1="111.76" y1="30.48" x2="152.4" y2="30.48" width="0.1524" layer="91"/>
 <wire x1="152.4" y1="30.48" x2="152.4" y2="20.32" width="0.1524" layer="91"/>
-<pinref part="J1" gate="G$1" pin="VCC"/>
+<pinref part="J1[SIMCARD]" gate="G$1" pin="VCC"/>
 <wire x1="152.4" y1="20.32" x2="147.32" y2="20.32" width="0.1524" layer="91"/>
 <wire x1="152.4" y1="30.48" x2="157.48" y2="30.48" width="0.1524" layer="91"/>
@@
 <wire x1="162.56" y1="-10.16" x2="162.56" y2="10.16" width="0.1524" layer="91"/>
 <wire x1="162.56" y1="10.16" x2="147.32" y2="10.16" width="0.1524" layer="91"/>
-<pinref part="J1" gate="G$1" pin="I/O"/>
+<pinref part="J1[SIMCARD]" gate="G$1" pin="I/O"/>
 <pinref part="D4" gate="1" pin="C"/>
 <junction x="93.98" y="5.08"/>
@@
 </segment>
 <segment>
-<pinref part="J3" gate="G$1" pin="1"/>
+<pinref part="J3[GROVE]" gate="G$1" pin="1"/>
 <wire x1="190.5" y1="20.32" x2="190.5" y2="27.94" width="0.1524" layer="91"/>
 <wire x1="190.5" y1="27.94" x2="195.58" y2="27.94" width="0.1524" layer="91"/>
@@
 <net name="N$9" class="0">
 <segment>
-<pinref part="J3" gate="G$1" pin="2"/>
+<pinref part="J3[GROVE]" gate="G$1" pin="2"/>
 <pinref part="R7" gate="G$1" pin="1"/>
 <wire x1="190.5" y1="17.78" x2="182.88" y2="17.78" width="0.1524" layer="91"/>
@@
 <net name="N$10" class="0">
 <segment>
-<pinref part="J3" gate="G$1" pin="3"/>
+<pinref part="J3[GROVE]" gate="G$1" pin="3"/>
 <wire x1="190.5" y1="15.24" x2="172.72" y2="15.24" width="0.1524" layer="91"/>
 <pinref part="R8" gate="G$1" pin="1"/>

Commit message: Schematic & Layout Updates
Updates made prior to poster publishing for Demo Day Poster!
Parts:
- removed D4, D5, D6, D7: 1N4004, diode:1N4004
- added C7: 0.1uF, capacitor-wima:C2,5-3
- added J4[GROVE]: 640456-4, 640456-4:640456-4
- added R11, R12, R13, R14, R15, R16: (no value), SparkFun-Resistors:RESISTOR0402
- added SV1, SV2: (no value), con-lstb:MA18-2
- added SW2, SW3: (no value), adafruit:SWITCH_PUSHBUTTONSOFTTOUCHSMD_SJ
- added U$1: MSQA6V1W5T2G, Personal:MSQA6V1W5T2G
- added U2: TUSB2046BIRHBR, TUSB2046B:TUSB2046BIRHBR
- SW1: value CT10-XXXX-A2 -> (none); device switch-coto:CT10-XXXX-A2 -> adafruit:SWITCH_PUSHBUTTONSOFTTOUCHSMD_SJ
Connections:
- new net N$12: J4[GROVE].2, R11.1
- new net N$13: J4[GROVE].3, R12.1
- new net N$14: R13.1, SW2.P$2
- new net N$15: R15.1, SW3.P$2
- net +5V: now also C7.2, J4[GROVE].1, R11.2, R12.2, R13.2, R15.2
- net 0: now also C7.1, J4[GROVE].4, R14.1, R16.1, U$1.P$2; no longer D4.A, D5.A, D6.A, D7.A
- net N$1: now also C6.1, J1[SIMCARD].VCC, U$1.P$5, U1.SIM_VDD; no longer J1[SIMCARD].RST, U1.SIM_CLK
- net N$11: now also SW1.P$2; no longer SW1.2
- net N$2: now also U$1.P$3; no longer D5.C, D6.C
- net N$4: now also J1[SIMCARD].RST, U$1.P$1, U1.SIM_CLK; no longer C6.1, D7.C, J1[SIMCARD].VCC, U1.SIM_VDD
- net N$6: now also U$1.P$4; no longer D4.C
- net NRESET: now also R14.2, R16.2, SW1.P$1, SW2.P$1, SW3.P$1; no longer SW1.1

Commit message: PCB Review 2 meeting Push
Parts:
- removed J3[GROVE]: 640456-4, 640456-4:640456-4
- added C10, C11, C8, C9: (no value), rcl:C-USC0805
- added C12, C13, C14, C15: 27pF, rcl:C-USC0603
- added CR1: 9C-6.000MAAJ-T, Personal:9C-6.000MAAJ-T
- added D4: Yellow, SparkFun-LED:LED-YELLOW0603
- added GROVE1: 640456-4, 640456-4:640456-4
- added J1: AU-Y1008-2, Personal:AU-Y1008-2
- added R17: 4.7k, SparkFun-Resistors:4.7KOHM-0603-1/10W-1%
- added R18: 47k, SparkFun-Resistors:47KOHM-0603-1/10W-1%
- added R19, R20: 27, SparkFun-Resistors:RESISTOR0805
- added R21, R22: (no value), SparkFun-Resistors:RESISTOR0805
- added R23, R24: 15k, SparkFun-Resistors:RESISTOR0805
- added R25: 1.5k, SparkFun-Resistors:RESISTOR0805
- added R26, R27: 0, SparkFun-Resistors:1KOHM-0603-1/10W-1%
- added R28: 330, SparkFun-Resistors:1KOHM-0603-1/10W-1%
- added R29, R30, R31, R32: 4700, SparkFun-Resistors:RESISTOR0805
- added SJ1: (no value), jumper:SJ
- added T1, T2: BCX70SMD, transistor:BCX70SMD
- added TP1, TP10, TP11, TP12, TP13, TP14, TP15, TP16, TP17, TP18, TP19, TP3, TP4, TP5, TP6, TP7, TP8, TP9: TPTP10R, testpad:TPTP10R
- added TP2: TPTP16R, testpad:TPTP16R
- added U3: MAX3373EEKA+T, Personal:MAX3373EEKA+T
- added U4: TPS2044BDR, Personal:TPS2044BDR
- added X1: 332-04, con-garry:332-04
- C1, C2, C3, C6, C7: device capacitor-wima:C2,5-3 -> rcl:C-USC0805
- C4, C5: device rcl:C-US025-024X044 -> rcl:C-USC0805
- D1: value (none) -> RED; device SparkFun-LED:LED-3MM-NO_SILK -> SparkFun-LED:LED-RED1206
- D2: value (none) -> GREEN; device SparkFun-LED:LED-3MM-NO_SILK -> SparkFun-LED:LED-GREEN1206
- D3: value (none) -> BLUE; device SparkFun-LED:LED-3MM-NO_SILK -> SparkFun-LED:LED-BLUE1206
- J2: value 292303-1 -> U.FL-R-SMT-1(01); device 292303-1:292303-1 -> Personal:U.FL-R-SMT-1(01)
- R1, R2, R3: value (none) -> 330; device SparkFun-Resistors:RESISTOR0402 -> SparkFun-Resistors:RESISTOR0805
- R10, R14, R16, R4, R5, R6: device SparkFun-Resistors:RESISTOR0402 -> SparkFun-Resistors:RESISTOR0805
- R11: value (none) -> 47k; device SparkFun-Resistors:RESISTOR0402 -> SparkFun-Resistors:47KOHM-0603-1/10W-1%
- R12: value (none) -> 4.7k; device SparkFun-Resistors:RESISTOR0402 -> SparkFun-Resistors:4.7KOHM-0603-1/10W-1%
- R13, R15: value (none) -> 15k; device SparkFun-Resistors:RESISTOR0402 -> SparkFun-Resistors:RESISTOR0805
- R7, R8: value (none) -> 27; device SparkFun-Resistors:RESISTOR0402 -> SparkFun-Resistors:RESISTOR0805
- R9: value (none) -> 1.5k; device SparkFun-Resistors:RESISTOR0402 -> SparkFun-Resistors:1KOHM-0603-1/10W-1%
- U2: value TUSB2046BIRHBR -> TUSB2046BVFR; device TUSB2046B:TUSB2046BIRHBR -> Personal:TUSB2046BVFR
- renumbered IC1 to POWER_SUPPLY
Connections:
- removed net 0: C1.2, C2.1, C3.2, C4.2, C5.2, C6.2, C7.1, D1.A, D2.A, D3.A, J1[SIMCARD].GND, J2.P4, J3[GROVE].4, J4[GROVE].4, POWER_SUPPLY.GND, R10.1, R14.1, R16.1, R4.1, R6.1, U$1.P$2, U1.GND
- removed net GPIO_1: R3.2
- removed net GPIO_2: R2.2
- removed net GPIO_3: R1.2
- removed net UART_RXD: U1.RXD
- removed net UART_TXD: U1.TXD
- removed net VBAT: C3.1, C5.1, POWER_SUPPLY.OUT, R5.2, R6.2, U1.VBAT
- removed net WIFI_D+: J2.P3
- removed net WIFI_D-: J2.P2
- new net 1.8V: C9.1, U1.VDD_EXT, U3.!THREESTATE, U3.VL
- new net 3.3V: C10.1, GROVE1.3, J4[GROVE].3, R17.2, R25.2, R29.2, R30.2, R31.2, R32.2, SJ1.1, SV1.14, U2.!EXTMEM, U2.VCC, U2.VCC_2, X1-1.S
- new net DM0: R8.1, SV1.9
- new net DP0: R7.1, SV1.11
- new net GND: C1.2, C10.2, C11.2, C12.2, C13.2, C14.2, C15.2, C2.1, C3.2, C4.2, C5.2, C6.2, C7.1, C8.2, C9.2, D1.C, D2.C, D3.C, D4.C, GROVE1.4, J1.4, J1.8, J1[SIMCARD].GND, J2.1, J2.3, J4[GROVE].4, POWER_SUPPLY.GND, R10.1, R11.2, R13.1, R14.1, R15.1, R16.1, R18.1, R23.1, R24.1, R4.1, R6.1, SV1.15, SV2.15, T1.E, T2.E, U$1.P$2, U1.GND, U2.BUSPWR, U2.EEDATA/GANGED, U2.GND, U2.GND_2, U2.TSTMODE, U2.TSTPLL/48MCLK, U3.GND, U3.VCC, U4.GND, U4.GND_2, X1-4.S
- new net I2C1_SCL: C2.2, GROVE1.1, R29.1, SV2.9, TP11.TP
- new net I2C1_SDA: GROVE1.2, R30.1, SV2.11, TP12.TP
- new net I2C2_SCL: C7.2, J4[GROVE].1, R31.1, SV1.28, TP13.TP
- new net I2C2_SDA: J4[GROVE].2, R32.1, SV1.26, TP14.TP
- new net LED1: R3.2, SV2.6
- new net LED2: R2.2, SV2.8
- new net LED3: R1.2, SV2.10
- new net MODEM_POWER: C3.1, C5.1, POWER_SUPPLY.OUT, R5.2, R6.2, SJ1.2, TP5.TP, U1.VBAT
- new net N$16: U3.IO/VL1, X1-3.S
- new net N$17: R11.1, R12.2, T2.B
- new net N$18: R17.1, R18.2, T1.B
- new net N$19: R19.2, U2.DM2
- new net N$20: R20.2, U2.DP2
- new net N$22: R21.1, U2.DP3
- new net N$23: R22.1, U2.DM3
- new net N$24: TP17.TP, U1.I2C_SCL
- new net N$25: U2.DP4
- new net N$26: U2.DM4
- new net N$27: TP16.TP, U1.RXD, U3.IO/VCC2
- new net N$28: TP15.TP, U1.TXD, U3.IO/VL2
- new net N$29: R28.2, U1.NETLIGHT
- new net N$30: D4.A, R28.1
- new net N$31: TP18.TP, U1.I2C_SDA
- new net OUT1: U4.OUT1
- new net OUT2: J1.1, TP3.TP, U4.OUT2
- new net OUT3: J1.5, TP4.TP, U4.OUT3
- new net OUT4: U4.NC
- new net OVRCUR1: U2.!OVRCUR1, U4.!OC1
- new net OVRCUR2: U2.!OVRCUR2, U4.!OC2
- new net OVRCUR3: U2.!OVRCUR3, U4.!OC3
- new net OVRCUR4: U2.!OVRCUR4, U4.NC_3
- new net PB2: R14.2, SV2.17, SW2.P$1
- new net PB3: R16.2, SV2.19, SW3.P$1
- new net PRE_ANT: C15.1, R26.2, U1.RF_ANT
- new net PWRKEY: C8.1, SV2.3, T1.C, U1.!PWRKEY
- new net PWRON1: U2.!PWRON1, U4.!EN1
- new net PWRON2: U2.!PWRON2, U4.!EN2
- new net PWRON3: U2.!PWRON3, U4.!EN3
- new net PWRON4: U2.!PWRON4, U4.NC_2
- new net RF_ANT: J2.2, R27.1
- new net SLEEP: R12.1, SV2.2
- new net USB1_D+: J1.3, R20.1, R24.2, TP8.TP
- new net USB1_D-: J1.2, R19.1, R23.2, TP7.TP
- new net USB2_D+: J1.7, R13.2, R21.2, TP10.TP
- new net USB2_D-: J1.6, R15.2, R22.2, TP9.TP
- new net VDD_EXT: T2.C, U1.DTR
- new net XTAL1: C12.1, CR1.1, U2.XTAL1
- new net XTAL2: R9.2, U2.XTAL2
- net +5V: now also C11.1, POWER_SUPPLY.EN, SV1.24, SW1.P$2, SW2.P$2, SW3.P$2, TP6.TP, U4.IN1, U4.IN2; no longer C2.2, C7.2, J2.P1, J3[GROVE].1, J4[GROVE].1, R11.2, R12.2, R13.2, R15.2, R7.2, R8.2, R9.2
- net MODEM_D+: now also U2.DP1
- net MODEM_D-: now also U2.DM1
- net N$10: now also R25.1, R7.2, U2.DP0; no longer J3[GROVE].3, R8.1
- net N$11: now also C14.1, R26.1, R27.2; no longer R9.1, SW1.P$2
- net N$12: now also R8.2, U2.DM0; no longer J4[GROVE].2, R11.1
- net N$13: now also U3.IO/VCC1, X1-2.S; no longer J4[GROVE].3, R12.1
- net N$14: now also C13.1, CR1.2, R9.1; no longer R13.1, SW2.P$2
- net N$15: now also TP2.TP, U1.GNSS_ANT; no longer R15.1, SW3.P$2
- net N$5: now also D3.A; no longer D3.C
- net N$6: now also TP19.TP
- net N$7: now also D2.A; no longer D2.C
- net N$8: now also D1.A; no longer D1.C
- net N$9: now also TP1.TP, U1.BOOT_CFG; no longer J3[GROVE].2, R7.1
- net NRESET: no longer R14.2, R16.2, SW2.P$1, SW3.P$1
Other:
- moved on the sheet: BRD1, C6, J1[SIMCARD], SV1, SV2, U1

Commit message: Hopefully Final Changes Pre-Alpha Purchase
*Still need to generate GERBERS*
Parts:
- added C16: 33pF, rcl:C-EUC0603K
- added J3: U.FL-R-SMT-1(01), Personal:U.FL-R-SMT-1(01)
- added L1: 47nH, rcl:C-EUC1608
- added TP20, TP21, TP22, TP23, TP24, TP25, TP26, TP27, TP28: TPTP10R, testpad:TPTP10R
Connections:
- removed net RF_ANT: J2.2, R27.1
- new net N$21: TP21.TP, U1.CTS
- new net N$32: TP22.TP, U1.RTS
- new net N$33: TP20.TP, U1.STATUS
- new net N$34: TP25.TP, U2.!RESET
- new net N$35: J2.3, R27.1
- new net N$36: C16.1, J3.3, L1.2
- net GND: now also C16.2, J2.2, J3.1, J3.2, TP26.TP, TP27.TP, TP28.TP; no longer J2.3
- net MODEM_POWER: now also L1.1
- net N$25: now also TP23.TP
- net N$26: now also TP24.TP

Commit message: Added team names to pcb and created gerber files
Other:
- note added: "Janak Patel Liza Lance Arthur Brazzle Alex Minser"
- note added: "NSCU ECE Senior Design 2020"
Changed lines of the file:
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@@
 <?xml version="1.0" encoding="utf-8"?>
 <!DOCTYPE eagle SYSTEM "eagle.dtd">
-<eagle version="9.6.2">
+<eagle version="9.6.0">
 <drawing>
 <settings>
-<setting alwaysvectorfont="yes"/>
+<setting alwaysvectorfont="no"/>
 <setting verticaltext="up"/>
 </settings>
@@
 <sheet>
 <plain>
+<text x="-68.58" y="-127" size="1.778" layer="112">NSCU ECE Senior Design 2020</text>
+<text x="-60.96" y="-137.16" size="1.778" layer="112">Janak Patel
+Liza Lance
+Arthur Brazzle
+Alex Minser</text>
 </plain>
 <instances>
@@
 </drawing>
 <compatibility>
+<note version="6.3" minversion="6.2.2" severity="warning">
+Since Version 6.2.2 text objects can contain more than one line,
+which will not be processed correctly with this version.
+</note>
 <note version="8.2" severity="warning">
 Since Version 8.2, EAGLE supports online libraries. The ids
